File: projects/uext-breadboard.sch (KiCad schematic (older format))
At the start: 6 parts, among them CON1 UEXT-5V, CON2 UEXT-BREADBOARD, CON3 UEXT-5V, U1 LM1117-3.3

Commit message: added latest projects
Parts:
- added C3: CP, Capacitors_THT:CP_Radial_D8.0mm_P5.00mm, symbol CP
- added J1: CONN_01X11, Pin_Headers:Pin_Header_Straight_1x11_Pitch2.54mm, symbol CONN_01X11
- C1: footprint Capacitors_THT:CP_Axial_L10.0mm_D6.0mm_P15.00mm_Horizontal -> Capacitors_THT:CP_Radial_D8.0mm_P5.00mm
- C2: footprint Capacitors_THT:C_Axial_L5.1mm_D3.1mm_P7.50mm_Horizontal -> Capacitors_THT:C_Disc_D8.0mm_W5.0mm_P5.00mm
Connections:
- net labels added: MISO, MOSI, RXD, SCK, SCL, SDA, SSEL, TXD
- wire segments 20 -> 47
Other:
- moved on the sheet: CON2, CON3
Changed lines of the file:
@@
 LIBS:contrib
 LIBS:valves
-LIBS:nodemcu
-LIBS:uext
 LIBS:limero
-LIBS:uext-breadboard-cache
 EELAYER 25 0
 EELAYER END
@@
 $EndDescr
 $Comp
-L UEXT-BREADBOARD CON2
-U 1 1 59711C4F
-P 5800 2550
-F 0 "CON2" H 5400 2250 40  0000 C CNN
-F 1 "UEXT-BREADBOARD" H 5950 2250 40  0000 C CNN
-F 2 "limero-lib:UEXT-BREADBOARD" H 5500 2550 60  0001 C CNN
-F 3 "" H 5500 2550 60  0000 C CNN
-	1    5800 2550
-	1    0    0    -1
-$EndComp
-$Comp
 L LM1117-3.3 U1
 U 1 1 59711F8A
@@
 F 0 "C1" H 4025 3000 50  0000 L CNN
 F 1 "CP" H 4025 2800 50  0000 L CNN
-F 2 "Capacitors_THT:CP_Axial_L10.0mm_D6.0mm_P15.00mm_Horizontal" H 4038 2750 50  0001 C CNN
+F 2 "Capacitors_THT:CP_Radial_D8.0mm_P5.00mm" H 4038 2750 50  0001 C CNN
 F 3 "" H 4000 2900 50  0001 C CNN
 	1    4000 2900
@@
 F 0 "C2" H 4375 3000 50  0000 L CNN
 F 1 "C" H 4375 2800 50  0000 L CNN
-F 2 "Capacitors_THT:C_Axial_L5.1mm_D3.1mm_P7.50mm_Horizontal" H 4388 2750 50  0001 C CNN
+F 2 "Capacitors_THT:C_Disc_D8.0mm_W5.0mm_P5.00mm" H 4388 2750 50  0001 C CNN
 F 3 "" H 4350 2900 50  0001 C CNN
 	1    4350 2900
@@
 $EndComp
 Wire Wire Line
-	6250 2750 6600 2750
-Wire Wire Line
-	6250 2650 6600 2650
-Wire Wire Line
-	6250 2550 6600 2550
-Wire Wire Line
-	6250 2450 6600 2450
-Wire Wire Line
-	6250 2350 6600 2350
-Wire Wire Line
-	5450 2350 5100 2350
-Wire Wire Line
-	5450 2450 5100 2450
-Wire Wire Line
-	5450 2550 5100 2550
-Wire Wire Line
-	5100 2650 5450 2650
-Wire Wire Line
-	5450 2750 5100 2750
-Wire Wire Line
 	3000 2700 3200 2700
 Wire Wire Line
 	3500 3000 3500 3200
 Wire Wire Line
-	3500 3200 4350 3200
+	3000 3200 4350 3200
 Wire Wire Line
 	4000 3200 4000 3050
@@
 Connection ~ 4350 2700
 $Comp
-L UEXT-5V CON3
-U 1 1 59712B3F
-P 5850 2550
-F 0 "CON3" H 5700 2850 40  0000 C CNN
-F 1 "UEXT-5V" H 6000 2250 40  0000 C CNN
-F 2 "limero-lib:UEXT" H 5550 2550 60  0001 C CNN
-F 3 "" H 5550 2550 60  0000 C CNN
-	1    5850 2550
-	1    0    0    -1
-$EndComp
-$Comp
 L UEXT-5V CON1
 U 1 1 59712BEF
@@
 L GND #PWR05
 U 1 1 59712D2F
-P 4350 3750
-F 0 "#PWR05" H 4350 3500 50  0001 C CNN
-F 1 "GND" H 4350 3600 50  0000 C CNN
-F 2 "" H 4350 3750 50  0001 C CNN
-F 3 "" H 4350 3750 50  0001 C CNN
-	1    4350 3750
-	1    0    0    -1
-$EndComp
-Wire Wire Line
-	3950 3750 4350 3750
+P 4400 3700
+F 0 "#PWR05" H 4400 3450 50  0001 C CNN
+F 1 "GND" H 4400 3550 50  0000 C CNN
+F 2 "" H 4400 3700 50  0001 C CNN
+F 3 "" H 4400 3700 50  0001 C CNN
+	1    4400 3700
+	-1   0    0    1
+$EndComp
+$Comp
+L +5V #PWR06
+U 1 1 5971B2A4
+P 5450 3700
+F 0 "#PWR06" H 5450 3550 50  0001 C CNN
+F 1 "+5V" H 5450 3840 50  0000 C CNN
+F 2 "" H 5450 3700 50  0001 C CNN
+F 3 "" H 5450 3700 50  0001 C CNN
+	1    5450 3700
+	1    0    0    -1
+$EndComp
+$Comp
+L GND #PWR07
+U 1 1 5971B2C4
+P 5250 3750
+F 0 "#PWR07" H 5250 3500 50  0001 C CNN
+F 1 "GND" H 5250 3600 50  0000 C CNN
+F 2 "" H 5250 3750 50  0001 C CNN
+F 3 "" H 5250 3750 50  0001 C CNN
+	1    5250 3750
+	-1   0    0    1
+$EndComp
+Text GLabel 5650 3950 0    60   Input ~ 0
+TXD
+Text GLabel 5650 4050 0    60   Input ~ 0
+RXD
+Text GLabel 5650 4150 0    60   Input ~ 0
+SCL
+Text GLabel 5650 4250 0    60   Input ~ 0
+SDA
+Text GLabel 5700 4450 0    60   Input ~ 0
+MOSI
+Text GLabel 5700 4350 0    60   Input ~ 0
+MISO
+Text GLabel 5650 4550 0    60   Input ~ 0
+SCK
+Text GLabel 5700 4650 0    60   Input ~ 0
+SSEL
+$Comp
+L CONN_01X11 J1
+U 1 1 5971B947
+P 6100 4150
+F 0 "J1" H 6100 4750 50  0000 C CNN
+F 1 "CONN_01X11" V 6200 4150 50  0000 C CNN
+F 2 "Pin_Headers:Pin_Header_Straight_1x11_Pitch2.54mm" H 6100 4150 50  0001 C CNN
+F 3 "" H 6100 4150 50  0001 C CNN
+	1    6100 4150
+	1    0    0    -1
+$EndComp
+Wire Wire Line
+	5650 3950 5900 3950
+Wire Wire Line
+	5900 3950 5900 3900
+Wire Wire Line
+	5650 4050 5900 4050
+Wire Wire Line
+	5650 4150 5900 4150
+Wire Wire Line
+	5650 4250 5900 4250
+Wire Wire Line
+	5700 4350 5900 4350
+Wire Wire Line
+	5700 4450 5900 4450
+Wire Wire Line
+	5900 4450 5900 4400
+Wire Wire Line
+	5650 4550 5900 4550
+Wire Wire Line
+	5700 4650 5900 4650
+Text GLabel 2800 3850 0    60   Input ~ 0
+TXD
+Text GLabel 4400 3850 2    60   Input ~ 0
+RXD
+Text GLabel 2800 3950 0    60   Input ~ 0
+SCL
+Text GLabel 4400 3950 2    60   Input ~ 0
+SDA
+Text GLabel 2850 4050 0    60   Input ~ 0
+MISO
+Text GLabel 4400 4050 2    60   Input ~ 0
+MOSI
+Text GLabel 2800 4150 0    60   Input ~ 0
+SCK
+Text GLabel 4400 4150 2    60   Input ~ 0
+SSEL
+Wire Wire Line
+	2800 3850 3150 3850
+Wire Wire Line
+	2800 3950 3150 3950
+Wire Wire Line
+	2850 4050 3150 4050
+Wire Wire Line
+	2800 4150 3150 4150
+Wire Wire Line
+	3950 3850 4400 3850
+Wire Wire Line
+	3950 3950 4400 3950
+Wire Wire Line
+	3950 4050 4400 4050
+Wire Wire Line
+	3950 4150 4400 4150
+Wire Wire Line
+	3950 3750 4400 3750
+Wire Wire Line
+	4400 3750 4400 3700
+Wire Wire Line
+	5250 3750 5250 3850
+Wire Wire Line
+	5250 3850 5900 3850
+Wire Wire Line
+	5450 3700 5450 3750
+Wire Wire Line
+	5450 3750 5900 3750
+$Comp
+L +3V3 #PWR08
+U 1 1 5971C070
+P 5650 3650
+F 0 "#PWR08" H 5650 3500 50  0001 C CNN
+F 1 "+3V3" H 5650 3790 50  0000 C CNN
+F 2 "" H 5650 3650 50  0001 C CNN
+F 3 "" H 5650 3650 50  0001 C CNN
+	1    5650 3650
+	1    0    0    -1
+$EndComp
+Wire Wire Line
+	5650 3650 5900 3650
+$Comp
+L CP C3
+U 1 1 5971C216
+P 3000 2850
+F 0 "C3" H 3025 2950 50  0000 L CNN
+F 1 "CP" H 3025 2750 50  0000 L CNN
+F 2 "Capacitors_THT:CP_Radial_D8.0mm_P5.00mm" H 3038 2700 50  0001 C CNN
+F 3 "" H 3000 2850 50  0001 C CNN
+	1    3000 2850
+	1    0    0    -1
+$EndComp
+Wire Wire Line
+	3000 3000 3000 3200
+Connection ~ 3500 3200
+Wire Wire Line
+	5500 2400 5150 3100
+Wire Wire Line
+	5150 3000 5500 2300
+Wire Wire Line
+	5500 2200 5150 2900
+Wire Wire Line
+	5500 2100 5150 2800
+Wire Wire Line
+	5500 2000 5150 2700
+Wire Wire Line
+	6300 2000 6650 2700
+Wire Wire Line
+	6300 2100 6650 2800
+Wire Wire Line
+	6300 2200 6650 2900
+Wire Wire Line
+	6300 2300 6650 3000
+Wire Wire Line
+	6300 2400 6650 3100
+$Comp
+L UEXT-BREADBOARD CON2
+U 1 1 59711C4F
+P 5850 2900
+F 0 "CON2" H 5450 2600 40  0000 C CNN
+F 1 "UEXT-BREADBOARD" H 6000 2600 40  0000 C CNN
+F 2 "limero-lib:UEXT-BREADBOARD" H 5550 2900 60  0001 C CNN
+F 3 "" H 5550 2900 60  0000 C CNN
+	1    5850 2900
+	1    0    0    -1
+$EndComp
+$Comp
+L UEXT-5V CON3
+U 1 1 59712B3F
+P 5900 2200
+F 0 "CON3" H 5750 2500 40  0000 C CNN
+F 1 "UEXT-5V" H 6050 1900 40  0000 C CNN
+F 2 "limero-lib:UEXT" H 5600 2200 60  0001 C CNN
+F 3 "" H 5600 2200 60  0000 C CNN
+	1    5900 2200
+	1    0    0    -1
+$EndComp
+$Comp
+L GND #PWR09
+U 1 1 5971C476
+P 6550 2000
+F 0 "#PWR09" H 6550 1750 50  0001 C CNN
+F 1 "GND" H 6550 1850 50  0000 C CNN
+F 2 "" H 6550 2000 50  0001 C CNN
+F 3 "" H 6550 2000 50  0001 C CNN
+	1    6550 2000
+	-1   0    0    1
+$EndComp
+$Comp
+L +5V #PWR010
+U 1 1 5971C4A1
+P 5250 2000
+F 0 "#PWR010" H 5250 1850 50  0001 C CNN
+F 1 "+5V" H 5250 2140 50  0000 C CNN
+F 2 "" H 5250 2000 50  0001 C CNN
+F 3 "" H 5250 2000 50  0001 C CNN
+	1    5250 2000
+	1    0    0    -1
+$EndComp
+Wire Wire Line
+	5250 2000 5500 2000
+Wire Wire Line
+	6550 2000 6300 2000
 $EndSCHEMATC
