File: projects/limero/limero.kicad_pcb (KiCad board)
At the start: 2 copper layers, 3 parts, among them J1 CONN_02X09

Commit message: working on lawnmower
Parts:
- added J2: ATX24, Connectors_Molex:Molex_MiniFit-JR-5556-24A_2x12x4.20mm_Straight, F.Cu at (66.0, 86.4)
- added J3: ATX_24PIN, Connectors_Molex:Molex_MiniFit-JR-5556-24A_2x12x4.20mm_Straight, F.Cu at (66.0, 66.0)
- moved J1 63.8 mm to (85.1, 111.8)
- moved D2 46.1 mm to (102.9, 111.8)
- moved D1 45.6 mm to (102.9, 104.1)
Connections:
- J1 pad 16: (no net) -> Net-(J1-Pad16)
